Commit message: Modify the model

File: gcr5g_description/robots/gcr5g_description.urdf (robot description, URDF)
Before this commit: robot gcr5g_description, 20 links, 19 joints
Links:
- removed link world
- link Link3: mass 0.635358049167358 -> 0.63535804916724
- link Link3_1: mass 0.0375413118311207 -> 0.0375413118311208
- link Link4: mass 0.120753251857492 -> 0.120753251857373
- link Link5: mass 0.120753251793899 -> 0.120753251793781
- link Link6: mass 0.0609840111314347 -> 0.0609840111314345
- link Link_gripper: mass 0.149482825119315 -> 0.149482836163735
- link Link_gripper1: mass 0.00770136927180476 -> 0.00770136927180468
- link Link_gripper1_1: mass 0.00588778350213341 -> 0.00588778350213335
- link Link_gripper2: mass 0.00395321330648626 -> 0.0039532133064862
- link Link_gripper3: mass 0.00770136927180474 -> 0.0077013692718047
- link Link_gripper3_1: mass 0.00588778350213349 -> 0.00588778350213328
- link Link_gripper4: mass 0.00395321330648629 -> 0.00395321330648628
Joints:
- removed joint fixed
- joint Joint1: limit lower=-3.14 upper=3.14 effort=1 velocity=1 -> lower=-3 upper=3 effort=1 velocity=1
- joint Joint2: limit lower=-3.14 upper=0.5 effort=1 velocity=1 -> lower=-3.5 upper=0.5 effort=0 velocity=0
- joint Joint5: axis 0 0 1 -> 0 0 -1; origin xyz=0 0.0735 -0.02085 rpy=3.1416 0 3.1416 -> xyz=0 0.0735 -0.02085 rpy=0 0 0
- joint Joint6: limit lower=-3.14 upper=3.14 effort=1 velocity=1 -> lower=-3 upper=3 effort=1 velocity=1; origin xyz=0 0.02085 0.0735 rpy=3.1416 0 3.1416 -> xyz=0 0.02085 -0.0735 rpy=0 0 0
- joint Joint_gripper1: origin xyz=-0.0163 0.19555 0.0083 rpy=0 0 -1.5708 -> xyz=0.0163 0.19555 -0.0083 rpy=0 0 0
- joint Joint_gripper1_1: limit lower=-1.35 upper=1.35 effort=1 velocity=1 -> lower=-0.35 upper=0.35 effort=1 velocity=1; origin xyz=-0.05164 -0.01893 0.0017 rpy=0 0 0 -> xyz=0.01893 0.05164 -0.0017 rpy=0 0 -1.5708
- joint Joint_gripper2: origin xyz=-0.00738 0.21232 0.008 rpy=0 0 -1.5708 -> xyz=0.00738 0.21232 -0.008 rpy=0 0 -1.5708
- joint Joint_gripper3: origin xyz=0.0167 0.19555 0.0083 rpy=0 0 -1.5708 -> xyz=-0.0167 0.19555 -0.0083 rpy=0 0 -1.5708
- joint Joint_gripper3_1: origin xyz=-0.05164 0.01893 0.0017 rpy=0 0 0 -> xyz=-0.05164 -0.01893 -0.0017 rpy=0 0 0
- joint Joint_gripper4: origin xyz=0.00778 0.21232 0.008 rpy=0 0 -1.5708 -> xyz=-0.00778 0.21232 -0.008 rpy=0 0 -1.5708

Commit message: add line model

File: gcr5g_description/robots/gcr5g_description.urdf (robot description, URDF)
Before this commit: robot gcr5g_description, 19 links, 18 joints
Links:
- added link link_line, mass 1; collision box size=0.005 0.005 0.03; visual cylinder length=0.03 radius=0.005
Joints:
- added joint Joint_line: type fixed, parent Link6, child link_line, origin xyz=0 0.0525 0.055 rpy=0 0 0
